File: docs/Schematics/KiCad/TritonECU-Main/ADC.kicad_sch (KiCad schematic)
At the start: 0 parts

Commit message: Carrier: ADC sheet (ADS8588H, reference, HO2S buffers, knock, slow channels)
ADS8588H serial on DOUTA, +-10 V, external MAX6070AAUT25 gated by the new
ADC_REF_EN (PG10). MAF differential on ch 1, battery 180k/30k on pin 55,
VREF_5V on ch 8. HO2S x4 per o2-input-stage.md on OPA2376. Knock charge
amp on TLV9064, moved to +3.3 V with a 1.8 V VMID because it lands on a
3.3 V MCU ADC pin. DPFE, TFT, FP monitor conditioned for the MCU ADC.
Series R on the unbuffered channels fitted 0R pending [DECIDE].

gen_carrier_pcb.py: PACK groups placed by courtyard shelf packing.
gen_carrier.py: own dual/quad op-amp symbols, fills an empty placeholder
sheet and keeps its block uuid.

Co-Authored-By: Claude Opus 5.5 <noreply@anthropic.com>
Parts:
- added C801, C802, C803, C804, C806, C811, C812, C814, C815, C820, C825, C826, C832, C833, C837, C838: 100n, Capacitor_SMD:C_0603_1608Metric_Pad1.08x0.95mm_HandSolder, symbol Device:C
- added C805, C809, C810: 10u, Capacitor_SMD:C_0805_2012Metric_Pad1.18x1.45mm_HandSolder, symbol Device:C
- added C807, C808, C817, C819, C822, C824, C834, C835: 1u, Capacitor_SMD:C_0603_1608Metric_Pad1.08x0.95mm_HandSolder, symbol Device:C
- added C813: 4.7u, Capacitor_SMD:C_0805_2012Metric_Pad1.18x1.45mm_HandSolder, symbol Device:C
- added C816, C818, C821, C823: 1n, Capacitor_SMD:C_0603_1608Metric_Pad1.08x0.95mm_HandSolder, symbol Device:C
- added C827, C828: 220p, Capacitor_SMD:C_0603_1608Metric_Pad1.08x0.95mm_HandSolder, symbol Device:C
- added C829, C830: 620p, Capacitor_SMD:C_0603_1608Metric_Pad1.08x0.95mm_HandSolder, symbol Device:C
- added C831: 15n, Capacitor_SMD:C_0603_1608Metric_Pad1.08x0.95mm_HandSolder, symbol Device:C
- added C836: 10n, Capacitor_SMD:C_0603_1608Metric_Pad1.08x0.95mm_HandSolder, symbol Device:C
- added D801: SMBJ30A, Diode_SMD:D_SMB, symbol Device:D_TVS
- added D802, D803, D804, D806: BAT54S, Package_TO_SOT_SMD:SOT-23, symbol Diode:BAT54S
- added D805, D807, D810, D811: BAT54J, Diode_SMD:D_SOD-323F, symbol Device:D_Schottky
- added D808, D809: BAV199, Package_TO_SOT_SMD:SOT-23, symbol Diode:BAT54S
- added R801, R810, R811, R812, R813, R821, R825, R829, R833: 0, Resistor_SMD:R_0603_1608Metric_Pad0.98x0.95mm_HandSolder, symbol Device:R
- added R802, R803, R804, R805, R806, R807, R809, R841, R842, R843, R844, R847: 10k, Resistor_SMD:R_0603_1608Metric_Pad0.98x0.95mm_HandSolder, symbol Device:R
- added R808: 220, Resistor_SMD:R_0603_1608Metric_Pad0.98x0.95mm_HandSolder, symbol Device:R
- added R814, R815: 2.49k, Resistor_SMD:R_0603_1608Metric_Pad0.98x0.95mm_HandSolder, symbol Device:R
- added R816: 180k, Resistor_SMD:R_0603_1608Metric_Pad0.98x0.95mm_HandSolder, symbol Device:R
- added R817: 30k, Resistor_SMD:R_0603_1608Metric_Pad0.98x0.95mm_HandSolder, symbol Device:R
- added R818, R822, R826, R830: 10k, Resistor_SMD:R_0805_2012Metric_Pad1.20x1.40mm_HandSolder, symbol Device:R
- added R819, R823, R827, R831: 22M, Resistor_SMD:R_0805_2012Metric_Pad1.20x1.40mm_HandSolder, symbol Device:R
- added R820, R824, R828, R832, R836, R837, R839, R850: 1k, Resistor_SMD:R_0603_1608Metric_Pad0.98x0.95mm_HandSolder, symbol Device:R
- added R834: 91k, Resistor_SMD:R_0603_1608Metric_Pad0.98x0.95mm_HandSolder, symbol Device:R
- added R835: 9.1k, Resistor_SMD:R_0603_1608Metric_Pad0.98x0.95mm_HandSolder, symbol Device:R
- added R838, R840: 1M, Resistor_SMD:R_0603_1608Metric_Pad0.98x0.95mm_HandSolder, symbol Device:R
- added R845: 470, Resistor_SMD:R_0603_1608Metric_Pad0.98x0.95mm_HandSolder, symbol Device:R
- added R846: 100, Resistor_SMD:R_0603_1608Metric_Pad0.98x0.95mm_HandSolder, symbol Device:R
- added R848: 18k, Resistor_SMD:R_0603_1608Metric_Pad0.98x0.95mm_HandSolder, symbol Device:R
- added R849: 2.2k, Resistor_SMD:R_0603_1608Metric_Pad0.98x0.95mm_HandSolder, symbol Device:R
- added R851: 100k, Resistor_SMD:R_0603_1608Metric_Pad0.98x0.95mm_HandSolder, symbol Device:R
- added R852: 10.5k, Resistor_SMD:R_0603_1608Metric_Pad0.98x0.95mm_HandSolder, symbol Device:R
- added U801: ADS8588HIPM, Samacsys:QFP50P1200X1200X160-64N, symbol Samacsys:ADS8588HIPM
- added U802: MAX6070AAUT25+T, Package_TO_SOT_SMD:SOT-23-6, symbol Reference_Voltage:MAX6070AAUT25+T
- added U803, U804: OPA2376AQDRQ1, Package_SO:SOIC-8_3.9x4.9mm_P1.27mm, symbol TritonECU-Carrier:OPAMP2
- added U805: TLV9064QPWRQ1, Package_SO:TSSOP-14_4.4x5mm_P0.65mm, symbol TritonECU-Carrier:OPAMP4
- added U806: MAX6070AAUT18+T, Package_TO_SOT_SMD:SOT-23-6, symbol Reference_Voltage:MAX6070AAUT18+T
Connections:
- new net +3.3V: C806.1, C826.1, C832.1, D805.1 (K), D807.1 (K), D808.2 (K), D809.2 (K), D810.1 (K), D811.1 (K), R808.1, R849.1, U801.23 (DVDD), U801.6 (~{PAR}/SER/BYTE_SEL), U801.7 (~{STBY}), U801.8 (RANGE), U805.4 (V+), U806.3 (EN), U806.4 (VIN)
- new net +5V: C801.1, C802.1, C803.1, C804.1, C805.1, C815.1, C820.1, D802.2 (K), D803.2 (K), D804.2 (K), D806.2 (K), R834.1, U801.1 (AVDD_1), U801.37 (AVDD_2), U801.38 (AVDD_3), U801.48 (AVDD_4), U803.8 (V+), U804.8 (V+)
- new net ADC_BUSY: U801.14 (BUSY)
- new net ADC_CONVST: R801.1, U801.9 (CONVSTA)
- new net ADC_CONVSTB: R801.2, U801.10 (CONVSTB)
- new net ADC_CS: U801.13 (~{CS})
- new net ADC_DB0: R802.1, U801.16 (DB0)
- new net ADC_DB1: R803.1, U801.17 (DB1)
- new net ADC_DB11: R805.1, U801.29 (DB11)
- new net ADC_DB14: R806.1, U801.32 (DB14/HBEN)
- new net ADC_DB15: R807.1, U801.33 (DB15/BYTE_SEL)
- new net ADC_DB2: R804.1, U801.18 (DB2)
- new net ADC_MISO: U801.24 (DB7/DOUTA)
- new net ADC_REF: C813.1, C814.1, U801.42 (REFIN/REFOUT), U802.5 (OUTS), U802.6 (OUTF)
- new net ADC_REFCAP: C809.1, U801.44 (REFCAPA), U801.45 (REFCAPB)
- new net ADC_REF_EN: R809.1, U802.3 (EN)
- new net ADC_REF_FLT: C812.1, U802.1 (FILTER)
- new net ADC_REF_IN: C810.1, C811.1, R808.2, U802.4 (VIN)
- new net ADC_REGCAP1: C807.1, U801.36 (REGCAP1)
- new net ADC_REGCAP2: C808.1, U801.39 (REGCAP2)
- new net ADC_RESET: U801.11 (RESET)
- new net ADC_SCK: U801.12 (~{RD}/SCLK)
- new net CHT_A: R812.2, U801.57 (AIN_5P)
- new net CHT_IN: R812.1, R814.2
- new net DPFE: C836.1, D810.2 (A), R847.2, R848.1
- new net DPFE_IN: R847.1
- new net FP_MON: C838.1, R851.2, R852.1
- new net FP_MON_IN: R851.1
- new net GND: C801.2, C802.2, C803.2, C804.2, C805.2, C806.2, C807.2, C808.2, C809.2, C810.2, C811.2, C812.2, C813.2, C814.2, C815.2, C816.2, C817.2, C818.2, C819.2, C820.2, C821.2, C822.2, C823.2, C824.2, C825.2, C826.2, C831.2, C832.2, C833.2, C834.2, C835.2, C836.2, C837.2, C838.2, D801.2 (A2), D802.1 (A), D803.1 (A), D804.1 (A), D806.1 (A), D808.1 (A), D809.1 (A), R802.2, R803.2, R804.2, R805.2, R806.2, R807.2, R809.2, R817.2, R835.2, R848.2, R852.2, U801.2 (AGND_1), U801.26 (AGND_2), U801.3 (OS0), U801.34 (REFSEL), U801.35 (AGND_3), U801.4 (OS1), U801.40 (AGND_4), U801.41 (AGND_5), U801.43 (REFGND_1), U801.46 (REFGND_2), U801.47 (AGND_6), U801.5 (OS2), U801.52 (AIN_2GND), U801.54 (AIN_3GND), U801.56 (AIN_4GND), U801.58 (AIN_5GND), U801.60 (AIN_6GND), U801.62 (AIN_7GND), U801.64 (AIN_8GND), U802.2 (GND), U803.4 (V-), U804.4 (V-), U805.11 (V-), U806.2 (GND)
- new net IAT_A: R813.2, U801.59 (AIN_6P)
- new net IAT_IN: R813.1, R815.2
- new net KA_OUT: C827.2, R838.2, R841.1, U805.1 (OUT1)
- new net KB_OUT: C828.2, R840.2, R842.1, U805.7 (OUT2)
- new net KC_N: C829.1, R841.2, R843.1, U805.9 (-IN3)
- new net KC_P: C830.1, R842.2, R844.1, U805.10 (+IN3)
- new net KNK_FLT: C833.1, U806.1 (FILTER)
- new net KNOCK: C831.1, R845.2
- new net KNOCK_DIFF: C829.2, R843.2, R845.1, U805.8 (OUT3)
- new net KNOCK_IN: D808.3 (COM), R837.1
- new net KNOCK_RTN: D809.3 (COM), R839.1
- new net KN_IN: C828.1, R839.2, R840.1, U805.6 (-IN2)
- new net KP_IN: C827.1, R837.2, R838.1, U805.2 (-IN1)
- new net MAF_A: R810.2, U801.49 (AIN_1P)
- new net MAF_IN: R810.1
- new net MAF_RTN: U801.50 (AIN_1GND)
- new net O2_11_A: C819.1, R824.2, R825.2, U801.55 (AIN_4P)
- new net O2_11_IN: R822.1
- new net O2_12_IN: R826.1
- new net O2_1_BUF: R820.1, U803.1 (OUTA), U803.2 (-INA)
- new net O2_1_HZ: C816.1, D802.3 (COM), R818.2, R819.1, R821.1, U803.3 (+INA)
- new net O2_21_A: C817.1, R820.2, R821.2, U801.53 (AIN_3P)
- new net O2_21_IN: R818.1
- new net O2_22_IN: R830.1
- new net O2_2_BUF: R824.1, U803.6 (-INB), U803.7 (OUTB)
- new net O2_2_HZ: C818.1, D803.3 (COM), R822.2, R823.1, R825.1, U803.5 (+INB)
- new net O2_3_BUF: R828.1, U804.1 (OUTA), U804.2 (-INA)
- new net O2_3_HZ: C821.1, D804.3 (COM), R826.2, R827.1, R829.1, U804.3 (+INA)
- new net O2_4_BUF: R832.1, U804.6 (-INB), U804.7 (OUTB)
- new net O2_4_HZ: C823.1, D806.3 (COM), R830.2, R831.1, R833.1, U804.5 (+INB)
- new net O2_BIAS: R836.1
- new net O2_BIASNODE: C825.1, R819.2, R823.2, R827.2, R831.2, R834.2, R835.1, R836.2
- new net O2_DN1: C822.1, D805.2 (A), R828.2, R829.2
- new net O2_DN2: C824.1, D807.2 (A), R832.2, R833.2
- new net TFT: C837.1, D811.2 (A), R850.2
- new net TFT_IN: R849.2, R850.1
- new net TPS_A: R811.2, U801.51 (AIN_2P)
- new net TPS_IN: R811.1
- new net VBAT_A: R816.2, R817.1, U801.61 (AIN_7P)
- new net VBAT_SENSE: D801.1 (A1), R816.1
- new net VMID: C830.2, R844.2, U805.13 (-IN4), U805.14 (OUT4), U805.3 (+IN1), U805.5 (+IN2)
- new net VMID_F: C835.1, R846.2, U805.12 (+IN4)
- new net VREF_5V: R814.1, R815.1, U801.63 (AIN_8P)
- new net VREF_KNK: C834.1, R846.1, U806.5 (OUTS), U806.6 (OUTF)
- no-connect marks 0 -> 10
Other:
- note added: "10k pull-downs: DB0-2 per the AD7606C serial rule, DB15/BYTE SEL low = serial not byte mode, DB11/DB14 parked."
- note added: "ADC: ADS8588H, serial on DOUTA, RANGE high = +-10 V (forced: ch 8 is VREF at 5.00 V), OS0-2 low, external 2.5 V reference."
- note added: "Ch: 1 MAF diff (968 return on AIN1GND), 2 TPS, 3 HO2S 21, 4 HO2S 11 (buffered), 5 CHT, 6 IAT, 7 battery 180k/30k, 8 VREF_5V."
- note added: "EN gated by ADC_REF_EN, 10k pull-down holds it off in Standby. 25 ms wait after enable. REFSEL low = external."
- note added: "Guard each 22M node with a ring driven from the buffer output. Downstream pair: BAT54J to 3.3 V, the MCU ADC is 3.3 V."
- note added: "HO2S x4: 10k + 1n + BAT54S to +5V, 22M to the 455 mV bias node, OPA2376 follower, 1k + 1u after it. JP = 0R not fitted."
- note added: "Knock: TLV9064 differential charge amp. ON 3.3 V with VMID 1.8 V (MAX6070AAUT18), NOT 5 V / 2.5 V as drawn in"
- note added: "MCU ADC (3.3 V): DPFE 0-5 V via 10k/18k, TFT 2.2k pull-up from 3.3 V (tft-sensor.md), FP monitor 100k/10.5k"
- note added: "Reference: MAX6070AAUT25 on 3.3 V (EN threshold is 0.7 x VIN). 220R + 10u in, 0.1u FILTER, 4.7u + 100n at REFIN."
- note added: "Single GND net: AGND/PGND is a layout split at the star, not a schematic one."
- note added: "Unbuffered channels: series resistor footprints fitted 0R - review-analog-chain.md #4 is [DECIDE]. Thermistor"
- note added: "knock-front-end-schematic.md: KNOCK lands on PC3, a 3.3 V ADC. Cf 220p C0G, Rf 1M, R5-R8 0.1 % matched. Guard KP/KN_IN."
- note added: "like the solenoid supply sense. 1k into each pin + BAT54J to 3.3 V where the harness can reach the pin."
- note added: "pull-ups from VREF_5V (ratiometric with ch 8); value [CONFIRM] against Ford tables. Battery: no filter cap."
- title: (none) -> TritonECU carrier - ADC

Commit message: Carrier: Inputs sheet and switched rails for sleep
Inputs: one network per switch input - 4.7k pull-up to VPWR (ground-
switched only; VPWR so a TR bit closed in Park draws nothing parked),
SMF24A, 33k/15k, 10n, BAT54J to 3.3 V. TR1/2/4 and 4X4L ground-switched,
TR3A/BRAKE/ACP/TCS 12 V high-side. 4X4L mapped to EEC-V pin 14
(findings sec.14). IGN_WAKE from VPWR into PC13/WKUP4. TACH/SPEED bench
header, BOOT0 DFU solder jumper.

Switched rails: +5V and +3.3V stay up parked, so two TPS22917 load
switches on SW_RAIL_EN (PG12, 100k down) make +5V_SW / +3.3V_SW for the
running-only loads: 74HCT541 x3 and OE pull-ups, MAX9926 x3 and COUT
pull-ups, ADS8588H, OPA2376 x2, O2 bias, knock block, 74HC4051, TPS2H160B
FAULT pull-up, TFT pull-up. MCU, watchdog, CAN, SCP RX, clamps stay on.

gen_carrier_pcb.py: packer steps around existing parts, fills several
rects in turn, parks overflow below earlier parked parts.

Co-Authored-By: Claude Opus 5.5 <noreply@anthropic.com>
Connections:
- net +3.3V: no longer C806.1, C826.1, C832.1, D808.2 (K), D809.2 (K), R849.1, U801.23 (DVDD), U801.6 (~{PAR}/SER/BYTE_SEL), U801.7 (~{STBY}), U801.8 (RANGE), U805.4 (V+), U806.3 (EN), U806.4 (VIN)
- net +5V renamed +5V_SW
- new net +3.3V_SW: C806.1, C826.1, C832.1, D808.2 (K), D809.2 (K), R849.1, U801.23 (DVDD), U801.6 (~{PAR}/SER/BYTE_SEL), U801.7 (~{STBY}), U801.8 (RANGE), U805.4 (V+), U806.3 (EN), U806.4 (VIN)

Commit message: Carrier: AGND star, matched ADC returns, 6-layer route
- ADC core, reference and inputs move to a separate AGND net, joined to
  GND and SIGRTN only at NT801 (the star under EEC-V 91). TPS/CHT/IAT/VREF
  VxGND inputs return on SIGRTN.
- Matched 0R legs on AIN_nGND (R853-R856), R857 bleed and D812 clamp on
  MAF_G, per ADS8588H SBAS843A.
- PCB generator syncs schematic fields onto existing footprints and packs
  the ADC column so the AGND island stays clear of GND parts.
- Board goes to 6 layers (1.6 mm): F / In1 GND plane with AGND island /
  In2-In4 signal / B. route_carrier.py adds net classes, the plane,
  Freerouting DSN/SES export/import and a repair mode that pre-stitches
  GND/AGND pads to the plane. Freerouting plus hand routing: DRC 0
  errors, 0 unconnected, schematic parity clean (silkscreen still to tidy).

Co-Authored-By: Claude Opus 5.5 <noreply@anthropic.com>
Parts:
- added D812: BAV199, Package_TO_SOT_SMD:SOT-23, symbol Diode:BAT54S
- added NT801: NetTie_3, NetTie:NetTie-3_SMD_Pad0.5mm, symbol Device:NetTie_3
- added R853, R854, R855, R856: 0, Resistor_SMD:R_0603_1608Metric_Pad0.98x0.95mm_HandSolder, symbol Device:R
- added R857: 10k, Resistor_SMD:R_0603_1608Metric_Pad0.98x0.95mm_HandSolder, symbol Device:R
- C817, C819: Note X7R 16 V -> X7R 16 V, at the converter
Connections:
- net +5V_SW: now also D812.2 (K)
- net GND: now also NT801.1; no longer C801.2, C802.2, C803.2, C804.2, C805.2, C806.2, C807.2, C808.2, C809.2, C810.2, C811.2, C812.2, C813.2, C814.2, C817.2, C819.2, R802.2, R803.2, R804.2, R805.2, R806.2, R807.2, R809.2, R817.2, U801.2 (AGND_1), U801.26 (AGND_2), U801.3 (OS0), U801.34 (REFSEL), U801.35 (AGND_3), U801.4 (OS1), U801.40 (AGND_4), U801.41 (AGND_5), U801.43 (REFGND_1), U801.46 (REFGND_2), U801.47 (AGND_6), U801.5 (OS2), U801.52 (AIN_2GND), U801.54 (AIN_3GND), U801.56 (AIN_4GND), U801.58 (AIN_5GND), U801.60 (AIN_6GND), U801.62 (AIN_7GND), U801.64 (AIN_8GND), U802.2 (GND)
- net MAF_RTN: now also R853.1; no longer U801.50 (AIN_1GND)
- new net AGND: C801.2, C802.2, C803.2, C804.2, C805.2, C806.2, C807.2, C808.2, C809.2, C810.2, C811.2, C812.2, C813.2, C814.2, C817.2, C819.2, D812.1 (A), NT801.2, R802.2, R803.2, R804.2, R805.2, R806.2, R807.2, R809.2, R817.2, R857.2, U801.2 (AGND_1), U801.26 (AGND_2), U801.3 (OS0), U801.34 (REFSEL), U801.35 (AGND_3), U801.4 (OS1), U801.40 (AGND_4), U801.41 (AGND_5), U801.43 (REFGND_1), U801.46 (REFGND_2), U801.47 (AGND_6), U801.5 (OS2), U801.54 (AIN_3GND), U801.56 (AIN_4GND), U801.62 (AIN_7GND), U802.2 (GND)
- new net CHT_G: R855.2, U801.58 (AIN_5GND)
- new net IAT_G: R856.2, U801.60 (AIN_6GND)
- new net MAF_G: D812.3 (COM), R853.2, R857.1, U801.50 (AIN_1GND)
- new net SIGRTN: NT801.3, R854.1, R855.1, R856.1, U801.64 (AIN_8GND)
- new net TPS_G: R854.2, U801.52 (AIN_2GND)
Other:
- note added: "AGND: the ADS8588H, its reference and its input conditioning. Meets GND and SIGRTN only at NT801, the star"
- note added: "AIN_nGND legs (ADS8588H 7.3.2): series R matched to"
- note added: "BAV199 to AGND/+5V_SW, 10k so an open 968 reads 0."
- note added: "MAF_RTN is the only remote one (+-0.3 V operating):"
- note added: "the AIN_nP series R, fitted 0R alongside them."
- note added: "under EEC-V 91. TPS, CHT, IAT and VREF sense are measured against SIGRTN (VxGND), MAF against MAF_RTN."
- note removed: "Single GND net: AGND/PGND is a layout split at the star, not a schematic one."
