File: docs/Schematics/KiCad/TritonECU-Main/Vref.kicad_sch (KiCad schematic)
At the start: 30 parts, among them Q701 DMN6040SVTQ-7, Q702 DMN6040SVTQ-7, U701 NCV8772CDT504RKG, U702 TPS2H160BQPWPRQ1, U703 LM74700QDBVRQ1, U704 LM74700QDBVRQ1

Commit message: Carrier: Inputs sheet and switched rails for sleep
Inputs: one network per switch input - 4.7k pull-up to VPWR (ground-
switched only; VPWR so a TR bit closed in Park draws nothing parked),
SMF24A, 33k/15k, 10n, BAT54J to 3.3 V. TR1/2/4 and 4X4L ground-switched,
TR3A/BRAKE/ACP/TCS 12 V high-side. 4X4L mapped to EEC-V pin 14
(findings sec.14). IGN_WAKE from VPWR into PC13/WKUP4. TACH/SPEED bench
header, BOOT0 DFU solder jumper.

Switched rails: +5V and +3.3V stay up parked, so two TPS22917 load
switches on SW_RAIL_EN (PG12, 100k down) make +5V_SW / +3.3V_SW for the
running-only loads: 74HCT541 x3 and OE pull-ups, MAX9926 x3 and COUT
pull-ups, ADS8588H, OPA2376 x2, O2 bias, knock block, 74HC4051, TPS2H160B
FAULT pull-up, TFT pull-up. MCU, watchdog, CAN, SCP RX, clamps stay on.

gen_carrier_pcb.py: packer steps around existing parts, fills several
rects in turn, parks overflow below earlier parked parts.

Co-Authored-By: Claude Opus 5.5 <noreply@anthropic.com>
Connections:
- net +3.3V: no longer R704.1
- new net +3.3V_SW: R704.1
